Commit message: udpate make map

File: src/lio_sam/config/robot.urdf.xacro (robot description, xacro)
@@ -7,10 +7,4 @@
     <parent link="base_link"/>
     <child link="chassis_link" />
-    <origin xyz="0 0 0" rpy="0 0 0" />
-  </joint>
-  <link name="lidar_link"> </link>
-  <joint name="lidar_joint" type="fixed">
-    <parent link="base_link" />
-    <child link="lidar_link" />
     <origin xyz="0 0 0" rpy="0 0 0" />
   </joint>

Commit message: gnssで地図生成

File: src/lio_sam/config/robot.urdf.xacro (robot description, xacro)
@@ -21,9 +21,9 @@
     <origin xyz="0 0 0" rpy="0 0 0" />
   </joint>
-  <link name="navsat_link"> </link>
+  <link name="gps"> </link>
   <joint name="navsat_joint" type="fixed">
     <parent link="chassis_link" />
-    <child link="navsat_link" />
-    <origin xyz="0 0 0" rpy="0 0 0" />
+    <child link="gps" />
+    <origin xyz="0 -0.12 0" rpy="0 0 0" />
   </joint>
 </robot>

Commit message: Add files via upload

File: src/lio_sam/config/robot.urdf.xacro (robot description, xacro)
@@ -25,5 +25,5 @@
     <parent link="chassis_link" />
     <child link="gps" />
-    <origin xyz="0 -0.12 0" rpy="0 0 0" />
+    <origin xyz="0 0 0.84" rpy="0 0 0" />
   </joint>
 </robot>

Commit message: Add files via upload

File: src/lio_sam/config/robot.urdf.xacro (robot description, xacro)
@@ -25,5 +25,5 @@
     <parent link="chassis_link" />
     <child link="gps" />
-    <origin xyz="0 0 0.84" rpy="0 0 0" />
+    <origin xyz="0 0 0" rpy="0 0 0" />
   </joint>
 </robot>
